Commit message: Improved the turning fix, added a lidar launch file

File: src/waveshare_real/robot_description/lidar.xacro (robot description, xacro)
@@ -4,5 +4,5 @@
         <parent link="base_link"/>
         <child link="lidar_link"/>
-        <origin xyz="0.042 0.0 0.1" rpy="0 0 0"/>
+        <origin xyz="0.042 0.0 0.1" rpy="0 0 3.14159"/>
     </joint>
     <link name="lidar_link">

File: src/waveshare_real/robot_description/robot.urdf.xacro (robot description, xacro)
@@ -17,4 +17,11 @@
         <link name="${prefix}base_link">
         </link>
+        <link name="${prefix}base_footprint">
+        </link>
+        <joint name="${prefix}base_footprint_joint" type="fixed">
+            <parent link="${prefix}base_link"/>
+            <child link="${prefix}base_footprint"/>
+            <origin xyz="0 0 0" rpy="0 0 0"/>
+        </joint>
         <joint name="${prefix}chassis_joint" type="fixed">
             <parent link="${prefix}base_link"/>
