Commit message: Quite a lot of troubleshooting for the missing links on /tf

File: src/waveshare_real/robot_description/robot.urdf.xacro (robot description, xacro)
@@ -3,149 +3,130 @@
     <xacro:include filename="inertial_macros.xacro"/>
     <xacro:macro name="waveshare_real" params="prefix">
-    <material name="white">
-        <color rgba="1 1 1 1"/>
-    </material>
-    <material name="blue">
-        <color rgba="0.2 0.2 1 1"/>
-    </material>
-    <material name="orange">
-        <color rgba="1 0.3 0.1 1"/>
-    </material>
-    <link name="${prefix}base_link">
-    </link>
-    <joint name="${prefix}chassis_joint" type="fixed">
-        <parent link="base_link"/>
-        <child link="chassis_link"/>
-        <origin xyz="-0.043 0.0 -0.0063"/>
-    </joint>
-    <link name="${prefix}chassis_link">
-        <visual>
-            <origin xyz="0.0915 0.0 0.02735"/>
-            <geometry>
-                <box size="0.183 0.083 0.0547"/>
-            </geometry>
-            <material name="white"/>
-        </visual>
-        <collision>
-            <origin xyz="0.0915 0 0.02735"/>
-            <geometry>
-                <box size="0.183 0.083 0.0547"/>
-            </geometry>
-        </collision>
-        <xacro:inertial_box mass="0.66" x="0.183" y="0.083" z="0.0547">
-            <origin xyz="0.0915 0 0.02735" rpy="0 0 0"/>
-        </xacro:inertial_box>
-    </link>
-    <gazebo reference="${prefix}chassis_link">
-        <material>Gazebo/White</material>
-    </gazebo>
-    <joint name="${prefix}lrw_joint" type="continuous">
-        <parent link="base_link"/>
-        <child link="lrw_link"/>
-        <origin xyz="0.0 0.06275 0.0" rpy="-1.5708 0 0"/>
-        <axis xyz="0 0 1"/>
-    </joint>
-    <link name="${prefix}lrw_link">
-        <visual>
-            <geometry>
-                <cylinder length="0.0425" radius="0.04"/>
-            </geometry>
-            <material name="blue"/>
-        </visual>
-        <collision>
-            <geometry>
-                <cylinder radius="0.04" length="0.0425"/>
-            </geometry>
-        </collision>
-        <xacro:inertial_cylinder mass="0.05" length="0.0425" radius="0.04">
-            <origin xyz="0 0 0" rpy="0 0 0"/>
-        </xacro:inertial_cylinder>
-    </link>
-    <gazebo reference="${prefix}lrw_link">
-        <material>Gazebo/Blue</material>
-        <mu1 value="0.4"/>
-        <mu2 value="0.4"/>
-    </gazebo>
-    <joint name="${prefix}rrw_joint" type="continuous">
-        <parent link="base_link"/>
-        <child link="rrw_link"/>
-        <origin xyz="0.0 -0.06275 0.0" rpy="1.5708 0 0"/>
-        <axis xyz="0 0 -1"/>
-    </joint>
-    <link name="${prefix}rrw_link">
-        <visual>
-            <geometry>
-                <cylinder length="0.0425" radius="0.04"/>
-            </geometry>
-            <material name="blue"/>
-        </visual>
-        <collision>
-            <geometry>
-                <cylinder radius="0.04" length="0.0425"/>
-            </geometry>
-        </collision>
-        <xacro:inertial_cylinder mass="0.05" length="0.0425" radius="0.04">
-            <origin xyz="0 0 0" rpy="0 0 0"/>
-        </xacro:inertial_cylinder>
-    </link>
-    <gazebo reference="${prefix}rrw_link">
-        <material>Gazebo/Blue</material>
-        <mu1 value="0.4"/>
-        <mu2 value="0.4"/>
-    </gazebo>
-    <joint name="${prefix}lfw_joint" type="continuous">
-        <parent link="base_link"/>
-        <child link="lfw_link"/>
-        <origin xyz="0.097 0.06275 0.0" rpy="-1.5708 0 0"/>
-        <axis xyz="0 0 1"/>
-    </joint>
-    <link name="${prefix}lfw_link">
-        <visual>
-            <geometry>
-                <cylinder length="0.0425" radius="0.04"/>
-            </geometry>
-            <material name="orange"/>
-        </visual>
-        <collision>
-            <geometry>
-                <cylinder radius="0.04" length="0.0425"/>
-            </geometry>
-        </collision>
-        <xacro:inertial_cylinder mass="0.05" length="0.0425" radius="0.04">
-            <origin xyz="0 0 0" rpy="0 0 0"/>
-        </xacro:inertial_cylinder>
-    </link>
-    <gazebo reference="${prefix}lfw_link">
-        <material>Gazebo/Orange</material>
-        <mu1 value="0.4"/>
-        <mu2 value="0.4"/>
-    </gazebo>
-    <joint name="${prefix}rfw_joint" type="continuous">
-        <parent link="base_link"/>
-        <child link="rfw_link"/>
-        <origin xyz="0.097 -0.06275 0.0" rpy="1.5708 0 0"/>
-        <axis xyz="0 0 -1"/>
-    </joint>
-    <link name="${prefix}rfw_link">
-        <visual>
-            <geometry>
-                <cylinder length="0.0425" radius="0.04"/>
-            </geometry>
-            <material name="orange"/>
-        </visual>
-        <collision>
-            <geometry>
-                <cylinder radius="0.04" length="0.0425"/>
-            </geometry>
-        </collision>
-        <xacro:inertial_cylinder mass="0.05" length="0.0425" radius="0.04">
-            <origin xyz="0 0 0" rpy="0 0 0"/>
-        </xacro:inertial_cylinder>
-    </link>
-    <gazebo reference="rfw_link">
-        <material>Gazebo/Orange</material>
-        <mu1 value="0.4"/>
-        <mu2 value="0.4"/>
-    </gazebo>
+        <material name="white">
+            <color rgba="1 1 1 1"/>
+        </material>
+        <material name="blue">
+            <color rgba="0.2 0.2 1 1"/>
+        </material>
+        <material name="orange">
+            <color rgba="1 0.3 0.1 1"/>
+        </material>
+        <link name="${prefix}base_link">
+        </link>
+        <joint name="${prefix}chassis_joint" type="fixed">
+            <parent link="${prefix}base_link"/>
+            <child link="${prefix}chassis_link"/>
+            <origin xyz="-0.043 0.0 -0.0063"/>
+        </joint>
+        <link name="${prefix}chassis_link">
+            <visual>
+                <origin xyz="0.0915 0.0 0.02735"/>
+                <geometry>
+                    <box size="0.183 0.083 0.0547"/>
+                </geometry>
+                <material name="white"/>
+            </visual>
+            <collision>
+                <origin xyz="0.0915 0 0.02735"/>
+                <geometry>
+                    <box size="0.183 0.083 0.0547"/>
+                </geometry>
+            </collision>
+            <xacro:inertial_box mass="0.66" x="0.183" y="0.083" z="0.0547">
+                <origin xyz="0.0915 0 0.02735" rpy="0 0 0"/>
+            </xacro:inertial_box>
+        </link>
+        <link name="${prefix}lrw_link">
+            <visual>
+                <geometry>
+                    <cylinder length="0.0425" radius="0.04"/>
+                </geometry>
+                <material name="blue"/>
+            </visual>
+            <collision>
+                <geometry>
+                    <cylinder radius="0.04" length="0.0425"/>
+                </geometry>
+            </collision>
+            <xacro:inertial_cylinder mass="0.05" length="0.0425" radius="0.04">
+                <origin xyz="0 0 0" rpy="0 0 0"/>
+            </xacro:inertial_cylinder>
+        </link>
+        <joint name="${prefix}lrw_joint" type="continuous">
+            <parent link="${prefix}base_link"/>
+            <child link="${prefix}lrw_link"/>
+            <origin xyz="0.0 0.06275 0.0" rpy="-1.5708 0 0"/>
+            <axis xyz="0 0 1"/>
+            <dynamics damping="0.2"/>
+        </joint>
+        <link name="${prefix}rrw_link">
+            <visual>
+                <geometry>
+                    <cylinder length="0.0425" radius="0.04"/>
+                </geometry>
+                <material name="blue"/>
+            </visual>
+            <collision>
+                <geometry>
+                    <cylinder radius="0.04" length="0.0425"/>
+                </geometry>
+            </collision>
+            <xacro:inertial_cylinder mass="0.05" length="0.0425" radius="0.04">
+                <origin xyz="0 0 0" rpy="0 0 0"/>
+            </xacro:inertial_cylinder>
+        </link>
+        <joint name="${prefix}rrw_joint" type="continuous">
+            <parent link="${prefix}base_link"/>
+            <child link="${prefix}rrw_link"/>
+            <origin xyz="0.0 -0.06275 0.0" rpy="1.5708 0 0"/>
+            <axis xyz="0 0 -1"/>
+            <dynamics damping="0.2"/>
+        </joint>
+        <link name="${prefix}lfw_link">
+            <visual>
+                <geometry>
+                    <cylinder length="0.0425" radius="0.04"/>
+                </geometry>
+                <material name="orange"/>
+            </visual>
+            <collision>
+                <geometry>
+                    <cylinder radius="0.04" length="0.0425"/>
+                </geometry>
+            </collision>
+            <xacro:inertial_cylinder mass="0.05" length="0.0425" radius="0.04">
+                <origin xyz="0 0 0" rpy="0 0 0"/>
+            </xacro:inertial_cylinder>
+        </link>
+        <joint name="${prefix}lfw_joint" type="continuous">
+            <parent link="${prefix}base_link"/>
+            <child link="${prefix}lfw_link"/>
+            <origin xyz="0.097 0.06275 0.0" rpy="-1.5708 0 0"/>
+            <axis xyz="0 0 1"/>
+            <dynamics damping="0.2"/>
+        </joint>
+        <link name="${prefix}rfw_link">
+            <visual>
+                <geometry>
+                    <cylinder length="0.0425" radius="0.04"/>
+                </geometry>
+                <material name="orange"/>
+            </visual>
+            <collision>
+                <geometry>
+                    <cylinder radius="0.04" length="0.0425"/>
+                </geometry>
+            </collision>
+            <xacro:inertial_cylinder mass="0.05" length="0.0425" radius="0.04">
+                <origin xyz="0 0 0" rpy="0 0 0"/>
+            </xacro:inertial_cylinder>
+        </link>
+        <joint name="${prefix}rfw_joint" type="continuous">
+            <parent link="${prefix}base_link"/>
+            <child link="${prefix}rfw_link"/>
+            <origin xyz="0.097 -0.06275 0.0" rpy="1.5708 0 0"/>
+            <axis xyz="0 0 -1"/>
+            <dynamics damping="0.2"/>
+        </joint>
     </xacro:macro>
 </robot>

File: src/waveshare_real/robot_description/rover.urdf.xacro (robot description, xacro)
@@ -2,8 +2,7 @@
 <robot xmlns:xacro="http://www.ros.org/wiki/xacro" name="waveshare_rover">
     <xacro:arg name="prefix" default="" />
-    <xacro:include filename="robot.urdf.xacro"/>
+    <xacro:include filename="$(find waveshare_real)/robot.urdf.xacro"/>
     <xacro:include filename="$(find waveshare_real)/waveshare_real.ros2_control.xacro" />
     <xacro:waveshare_real prefix="$(arg prefix)" />
-    <xacro:waveshare_real_ros2_control
-        name="waveshare_real" prefix="$(arg prefix)" />
+    <xacro:waveshare_real_ros2_control name="waveshare_real" prefix="$(arg prefix)" />
 </robot>

File: src/waveshare_real/robot_description/waveshare_real.ros2_control.xacro (robot description, xacro)
@@ -3,18 +3,20 @@
     <xacro:macro name="waveshare_real_ros2_control" params="name prefix">
         <ros2_control name="${name}" type="system">
-        <hardware>
-            <plugin>waveshare_real/WaveShareHardware</plugin>
-            <param name="rear_left_wheel_name">rlw_joint</param>
-            <param name="rear_right_wheel_name">rrw_joint</param>
-            <param name="loop_rate">30</param>
-            <param name="device">/dev/ttyUSB0</param>
-            <param name="baud_rate">115200</param>
-            <param name="timeout_ms">1000</param>
-            <param name="enc_counts_per_rev">555</param>
-            <param name="pid_p">50</param>
-            <param name="pid_d">0</param>
-            <param name="pid_i">90</param>
-            <param name="pid_o">50</param>
-        </hardware>
+            <hardware>
+                <plugin>waveshare_real/WaveShareHardware</plugin>
+                <param name="rear_left_wheel_name">rlw_joint</param>
+                <param name="front_left_wheel_name">flw_joint</param>
+                <param name="rear_right_wheel_name">rrw_joint</param>
+                <param name="front_right_wheel_name">frw_joint</param>
+                <param name="loop_rate">30</param>
+                <param name="device">/dev/ttyUSB0</param>
+                <param name="baud_rate">115200</param>
+                <param name="timeout_ms">2000</param>
+                <param name="enc_counts_per_rev">2555</param>
+                <param name="pid_p">50</param>
+                <param name="pid_d">0</param>
+                <param name="pid_i">90</param>
+                <param name="pid_o">50</param>
+            </hardware>
             <joint name="${prefix}rlw_joint">
                 <command_interface name="velocity" />
@@ -27,4 +29,14 @@
                 <state_interface name="velocity" />
             </joint>
+            <joint name="${prefix}flw_joint">
+                <command_interface name="velocity" />
+                <state_interface name="position" />
+                <state_interface name="velocity" />
+            </joint>
+            <joint name="${prefix}frw_joint">
+                <command_interface name="velocity" />
+                <state_interface name="position" />
+                <state_interface name="velocity" />
+            </joint>
         </ros2_control>
     </xacro:macro>

Commit message: Some troubleshooting for /tf, and for getting the square angles right

File: src/waveshare_real/robot_description/robot.urdf.xacro (robot description, xacro)
@@ -11,4 +11,7 @@
         <material name="orange">
             <color rgba="1 0.3 0.1 1"/>
+        </material>
+        <material name="red">
+            <color rgba="1 0 0 1"/>
         </material>
         <link name="${prefix}base_link">

File: src/waveshare_real/robot_description/rover.urdf.xacro (robot description, xacro)
@@ -4,4 +4,5 @@
     <xacro:include filename="$(find waveshare_real)/robot.urdf.xacro"/>
     <xacro:include filename="$(find waveshare_real)/waveshare_real.ros2_control.xacro" />
+    <xacro:include filename="$(find waveshare_real)/lidar.xacro" />
     <xacro:waveshare_real prefix="$(arg prefix)" />
     <xacro:waveshare_real_ros2_control name="waveshare_real" prefix="$(arg prefix)" />

Commit message: Fixed the problem of not all the wheel joints being published to /tf

File: src/waveshare_real/robot_description/robot.urdf.xacro (robot description, xacro)
@@ -47,5 +47,5 @@
             </xacro:inertial_box>
         </link>
-        <link name="${prefix}lrw_link">
+        <link name="${prefix}rlw_link">
             <visual>
                 <geometry>
@@ -63,7 +63,7 @@
             </xacro:inertial_cylinder>
         </link>
-        <joint name="${prefix}lrw_joint" type="continuous">
+        <joint name="${prefix}rlw_joint" type="continuous">
             <parent link="${prefix}base_link"/>
-            <child link="${prefix}lrw_link"/>
+            <child link="${prefix}rlw_link"/>
             <origin xyz="0.0 0.06275 0.0" rpy="-1.5708 0 0"/>
             <axis xyz="0 0 1"/>
@@ -93,5 +93,5 @@
             <dynamics damping="0.2"/>
         </joint>
-        <link name="${prefix}lfw_link">
+        <link name="${prefix}flw_link">
             <visual>
                 <geometry>
@@ -109,12 +109,12 @@
             </xacro:inertial_cylinder>
         </link>
-        <joint name="${prefix}lfw_joint" type="continuous">
+        <joint name="${prefix}flw_joint" type="continuous">
             <parent link="${prefix}base_link"/>
-            <child link="${prefix}lfw_link"/>
+            <child link="${prefix}flw_link"/>
             <origin xyz="0.097 0.06275 0.0" rpy="-1.5708 0 0"/>
             <axis xyz="0 0 1"/>
             <dynamics damping="0.2"/>
         </joint>
-        <link name="${prefix}rfw_link">
+        <link name="${prefix}frw_link">
             <visual>
                 <geometry>
@@ -132,7 +132,7 @@
             </xacro:inertial_cylinder>
         </link>
-        <joint name="${prefix}rfw_joint" type="continuous">
+        <joint name="${prefix}frw_joint" type="continuous">
             <parent link="${prefix}base_link"/>
-            <child link="${prefix}rfw_link"/>
+            <child link="${prefix}frw_link"/>
             <origin xyz="0.097 -0.06275 0.0" rpy="1.5708 0 0"/>
             <axis xyz="0 0 -1"/>
